File: hardware/dimmer/eagle/history/Dimmer_Board_Rev_0.1.sch (EAGLE design)
At the start: 18 parts, among them IC1 MCP23008/SO, SW1 EC11B

Commit message: Cleaning up Sch
Other:
- note added: "GPIO Expander"
- note added: "I2C Port"
- note added: "Rotary Encoder"
- note added: "Switches"
- note added: "v0.1"
- note removed: "v1.0"
- moved on the sheet: C1, C2, C3, IC1, JP1, JP2, JP3, JP4, R1, R2, R3, R4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
